File: src/ncp5623c-breakout.brd (EAGLE design)
At the start: 18 x 10.6 mm, 7 parts, among them J1 PTH VERT MALE, J2 PTH VERT MALE, U1 NCP5623CMUTBG

Commit message: Update CAM files.
Parts:
- moved C1 0.10 mm to (2.80, 1.70)
- moved C3 0.10 mm to (2.80, 0.45)
- moved R1 0.10 mm to (2.80, -0.80)
Connections:
- net GND: now also U1.EP
Routing:
- added copper zone on layer 1, net GND
Other:
- board text added: "Rev 2"
- board text removed: "Rev 1"
