File: src/ncp5623c-breakout.sch (EAGLE design)
At the start: 7 parts, among them J1 PTH VERT MALE, J2 PTH VERT MALE, U1 NCP5623CMUTBG

Commit message: Update CAM files.
Other:
- moved on the sheet: U1
